File: boards/fanpico-0804/kicad/extra_fan_channel.kicad_sch (KiCad schematic)
At the start: 9 parts

Commit message: PCB version 1.2
Other:
- title: FanPico-0804 -> FanPico-0804 v1.2
Changed lines of the file:
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@@
   (paper "A4")
   (title_block
-    (title "FanPico-0804")
-    (date "2022-02-26")
+    (title "FanPico-0804 v1.2")
+    (date "2022-03-11")
     (company "Timo Kokkonen <tjko@iki.fi>")
-    (comment 3 "Fanpico firmware reference/prototype PCB.")
+    (comment 3 "Fanpico firmware reference PCB.")
   )
   (junction (at 147.32 121.92) (diameter 0) (color 0 0 0 0)

Commit message: New PCB revision v1.3
Parts:
- renumbered C27 to C21, C28 to C22, D32 to D23, D33 to D24, D34 to D25, JP9 to JP6, R45 to R36, R46 to R37, R47 to R38
Other:
- title: FanPico-0804 v1.2 -> FanPico-0804 v1.3
Changed lines of the file:
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@@
   (paper "A4")
   (title_block
-    (title "FanPico-0804 v1.2")
-    (date "2022-03-11")
+    (title "FanPico-0804 v1.3")
+    (date "2022-04-10")
     (company "Timo Kokkonen <tjko@iki.fi>")
     (comment 3 "Fanpico firmware reference PCB.")
@@
     (effects (font (size 1.27 1.27)) (justify right))
   )
-  (symbol (lib_id "power:GND") (at 147.32 148.59 0)
-    (in_bom yes) (on_board yes) (fields_autoplaced)
-    (property "Reference" "#PWR079" (id 0) (at 147.32 154.94 0)
+  (symbol (lib_id "power:GND") (at 147.32 148.59 0) (unit 1)
+    (in_bom yes) (on_board yes) (fields_autoplaced)
+    (property "Reference" "#PWR067" (id 0) (at 147.32 154.94 0)
       (effects (font (size 1.27 1.27)) hide)
     )
@@
     (pin "1")
   )
-  (symbol (lib_id "power:GND") (at 146.05 91.44 0)
-    (in_bom yes) (on_board yes) (fields_autoplaced)
-    (property "Reference" "#PWR078" (id 0) (at 146.05 97.79 0)
+  (symbol (lib_id "power:GND") (at 146.05 91.44 0) (unit 1)
+    (in_bom yes) (on_board yes) (fields_autoplaced)
+    (property "Reference" "#PWR066" (id 0) (at 146.05 97.79 0)
       (effects (font (size 1.27 1.27)) hide)
     )
@@
     (pin "1")
   )
-  (symbol (lib_id "power:+3.3V") (at 160.02 60.96 90)
-    (in_bom yes) (on_board yes) (fields_autoplaced)
-    (property "Reference" "#PWR080" (id 0) (at 163.83 60.96 0)
+  (symbol (lib_id "power:+3.3V") (at 160.02 60.96 90) (unit 1)
+    (in_bom yes) (on_board yes) (fields_autoplaced)
+    (property "Reference" "#PWR068" (id 0) (at 163.83 60.96 0)
       (effects (font (size 1.27 1.27)) hide)
     )
@@
     (pin "1")
   )
-  (symbol (lib_id "Device:C") (at 146.05 83.82 0)
-    (in_bom yes) (on_board yes) (fields_autoplaced)
-    (property "Reference" "C27" (id 0) (at 149.86 82.5499 0)
+  (symbol (lib_id "Device:C") (at 146.05 83.82 0) (unit 1)
+    (in_bom yes) (on_board yes) (fields_autoplaced)
+    (property "Reference" "C21" (id 0) (at 149.86 82.5499 0)
       (effects (font (size 1.27 1.27)) (justify left))
     )
@@
     (pin "2")
   )
-  (symbol (lib_id "Device:C") (at 167.64 125.73 0)
-    (in_bom yes) (on_board yes) (fields_autoplaced)
-    (property "Reference" "C28" (id 0) (at 171.45 124.4599 0)
+  (symbol (lib_id "Device:C") (at 167.64 125.73 0) (unit 1)
+    (in_bom yes) (on_board yes) (fields_autoplaced)
+    (property "Reference" "C22" (id 0) (at 171.45 124.4599 0)
       (effects (font (size 1.27 1.27)) (justify left))
     )
@@
     (pin "2")
   )
-  (symbol (lib_id "Device:R") (at 147.32 129.54 0)
-    (in_bom yes) (on_board yes) (fields_autoplaced)
-    (property "Reference" "R45" (id 0) (at 149.86 128.2699 0)
+  (symbol (lib_id "Device:R") (at 147.32 129.54 0) (unit 1)
+    (in_bom yes) (on_board yes) (fields_autoplaced)
+    (property "Reference" "R36" (id 0) (at 149.86 128.2699 0)
       (effects (font (size 1.27 1.27)) (justify left))
     )
@@
     (pin "2")
   )
-  (symbol (lib_id "Device:R") (at 166.37 67.31 180)
-    (in_bom yes) (on_board yes) (fields_autoplaced)
-    (property "Reference" "R46" (id 0) (at 168.91 66.0399 0)
+  (symbol (lib_id "Device:R") (at 166.37 67.31 180) (unit 1)
+    (in_bom yes) (on_board yes) (fields_autoplaced)
+    (property "Reference" "R37" (id 0) (at 168.91 66.0399 0)
       (effects (font (size 1.27 1.27)) (justify right))
     )
@@
     (pin "2")
   )
-  (symbol (lib_id "Jumper:Jumper_3_Bridged12") (at 101.6 121.92 90)
-    (in_bom yes) (on_board yes) (fields_autoplaced)
-    (property "Reference" "JP9" (id 0) (at 99.06 120.6499 90)
+  (symbol (lib_id "Jumper:Jumper_3_Bridged12") (at 101.6 121.92 90) (unit 1)
+    (in_bom yes) (on_board yes) (fields_autoplaced)
+    (property "Reference" "JP6" (id 0) (at 99.06 120.6499 90)
       (effects (font (size 1.27 1.27)) (justify left))
     )
@@
     (pin "3")
   )
-  (symbol (lib_id "Device:D") (at 179.07 125.73 270)
-    (in_bom yes) (on_board yes) (fields_autoplaced)
-    (property "Reference" "D34" (id 0) (at 181.61 124.4599 90)
+  (symbol (lib_id "Device:D") (at 179.07 125.73 270) (unit 1)
+    (in_bom yes) (on_board yes) (fields_autoplaced)
+    (property "Reference" "D25" (id 0) (at 181.61 124.4599 90)
       (effects (font (size 1.27 1.27)) (justify left))
     )
@@
     (pin "2")
   )
-  (symbol (lib_id "Device:D") (at 177.8 74.93 180)
-    (in_bom yes) (on_board yes) (fields_autoplaced)
-    (property "Reference" "D33" (id 0) (at 177.8 68.58 0))
+  (symbol (lib_id "Device:D") (at 177.8 74.93 180) (unit 1)
+    (in_bom yes) (on_board yes) (fields_autoplaced)
+    (property "Reference" "D24" (id 0) (at 177.8 68.58 0))
     (property "Value" "BAT54C" (id 1) (at 177.8 71.12 0))
     (property "Footprint" "Diode_SMD:D_SOT-23_ANK" (id 2) (at 177.8 74.93 0)
@@
     (pin "2")
   )
-  (symbol (lib_id "power:GND") (at 179.07 135.89 0)
-    (in_bom yes) (on_board yes) (fields_autoplaced)
-    (property "Reference" "#PWR081" (id 0) (at 179.07 142.24 0)
+  (symbol (lib_id "power:GND") (at 179.07 135.89 0) (unit 1)
+    (in_bom yes) (on_board yes) (fields_autoplaced)
+    (property "Reference" "#PWR069" (id 0) (at 179.07 142.24 0)
       (effects (font (size 1.27 1.27)) hide)
     )
@@
     (pin "1")
   )
-  (symbol (lib_id "Device:R") (at 167.64 46.99 90)
-    (in_bom yes) (on_board yes) (fields_autoplaced)
-    (property "Reference" "R47" (id 0) (at 167.64 40.64 90))
+  (symbol (lib_id "Device:R") (at 167.64 46.99 90) (unit 1)
+    (in_bom yes) (on_board yes) (fields_autoplaced)
+    (property "Reference" "R38" (id 0) (at 167.64 40.64 90))
     (property "Value" "680" (id 1) (at 167.64 43.18 90))
     (property "Footprint" "Resistor_SMD:R_0603_1608Metric_Pad0.98x0.95mm_HandSolder" (id 2) (at 167.64 48.768 90)
@@
     (pin "2")
   )
-  (symbol (lib_id "Device:LED") (at 147.32 139.7 90)
-    (in_bom yes) (on_board yes) (fields_autoplaced)
-    (property "Reference" "D32" (id 0) (at 151.13 140.0174 90)
+  (symbol (lib_id "Device:LED") (at 147.32 139.7 90) (unit 1)
+    (in_bom yes) (on_board yes) (fields_autoplaced)
+    (property "Reference" "D23" (id 0) (at 151.13 140.0174 90)
       (effects (font (size 1.27 1.27)) (justify right))
     )

Commit message: Cleanup schematic (no actual changes that affect PCB).
- Add labels to sub-pages so printed schematic is more readable.
- Rename FANx_PWM_READ to MBFANx_PWM_READ
- Rename FANx_TACHO_GEN to MBFANx_TACHO_GEN
- Use standard (KiCAD) footprints for the ICs (U1-U3)
Connections:
- net +3V3 renamed +3.3V
Other:
- note added: "(Extra) Fan Channel: ${SHEETNAME}"
Changed lines of the file:
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@@
   (title_block
     (title "FanPico-0804 v1.3")
-    (date "2022-04-10")
+    (date "2022-08-18")
     (company "Timo Kokkonen <tjko@iki.fi>")
     (comment 3 "Fanpico firmware reference PCB.")
@@
     (effects (font (size 1.27 1.27)) (justify left bottom))
   )
+  (text "(Extra) Fan Channel: ${SHEETNAME}" (at 17.78 17.78 0)
+    (effects (font (size 2 2)) (justify left bottom))
+  )
   (text "To Fan" (at 209.55 35.56 0)
