File: boards/fanpico-0804/kicad/fanpico.kicad_sch (KiCad schematic)
At the start: 27 parts, among them J16 Sensor1, J17 Sensor2, J2 Pico Debug, J3 Floppy Power Connector, SW1 SW_Push, U1 SN74AHCT125QDRQ1, U2 SN74AHCT125QDRQ1, U3 CD74HC4050NSR, U4 Pico, U6 LM4040DBZ-3

Commit message: PCB version 1.2
Parts:
- removed J16: Sensor1, Connector_JST:JST_PH_B2B-PH-K_1x02_P2.00mm_Vertical, symbol Connector_Generic:Conn_01x02
- removed J17: Sensor2, Connector_JST:JST_PH_B2B-PH-K_1x02_P2.00mm_Vertical, symbol Connector_Generic:Conn_01x02
- removed R50, R51: 10k, Resistor_SMD:R_0603_1608Metric_Pad0.98x0.95mm_HandSolder, symbol Device:R
- C30: value 10uF 15V -> 10uF 16V; footprint Capacitor_SMD:C_1206_3216Metric_Pad1.33x1.80mm_HandSolder -> Capacitor_Tantalum_SMD:CP_EIA-3216-18_Kemet-A_Pad1.58x1.35mm_HandSolder
- R48: value 300 -> 330
- U1, U2: footprint Package_SO:SOIC-14_3.9x8.7mm_P1.27mm -> SOP65P640X120-14N
- U3: footprint Package_SO:SOP-16_3.9x9.9mm_P1.27mm -> SOIC127P600X175-16N
- U4: footprint MCU_RaspberryPi_and_Boards:RPi_Pico_SMD_TH -> RPi_Pico:RPi_Pico_SMD_TH
Other:
- added sheet Sensors (sensors.kicad_sch)
- note added: "3.3V to 5V TTL level converters (Outputs)"
- note added: "5-12V to 3.3V TTL level converters (Inputs)"
- note added: "Voltage Reference (ADC)"
- note removed: "3.3V to 5V level converters (Outputs)"
- note removed: "5-12V to 3.3V level converters (Inputs)"
- note removed: "Temperature Sensors"
- note removed: "Voltage Reference"
- title: FanPico-0804 -> FanPico-0804 v1.2
- moved on the sheet: C1, C2, C29, C3, C30, C4, D1, H1, H2, H3, H4, J2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

Commit message: New PCB revision v1.3
Parts:
- SW1: footprint Button_Switch_THT:SW_PUSH_6mm -> Button_Switch_THT:SW_PUSH_6mm_SMD_2
Other:
- title: FanPico-0804 v1.2 -> FanPico-0804 v1.3
Changed lines of the file:
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@@
   (paper "A4")
   (title_block
-    (title "FanPico-0804 v1.2")
-    (date "2022-03-11")
+    (title "FanPico-0804 v1.3")
+    (date "2022-04-10")
     (company "Timo Kokkonen <tjko@iki.fi>")
     (comment 3 "Fanpico firmware reference PCB.")
@@
     (property "Reference" "SW1" (id 0) (at 271.78 54.61 0))
     (property "Value" "SW_Push" (id 1) (at 271.78 57.15 0))
-    (property "Footprint" "Button_Switch_THT:SW_PUSH_6mm" (id 2) (at 271.78 57.15 0)
+    (property "Footprint" "Button_Switch_THT:SW_PUSH_6mm_SMD_2" (id 2) (at 271.78 57.15 0)
       (effects (font (size 1.27 1.27)) hide)
     )
@@
     )
     (path "/21c2b408-da95-4394-b5b2-e408611b3d07"
-      (reference "SW1") (unit 1) (value "SW_Push") (footprint "Button_Switch_THT:SW_PUSH_6mm")
+      (reference "SW1") (unit 1) (value "SW_Push") (footprint "Button_Switch_THT:SW_PUSH_6mm_SMD_2")
     )
     (path "/20cc4b05-e726-4b05-ab1c-64b5db072e26/146a1d06-dd1a-482f-b91e-93cbb733b8f4"

Commit message: Cleanup schematic (no actual changes that affect PCB).
- Add labels to sub-pages so printed schematic is more readable.
- Rename FANx_PWM_READ to MBFANx_PWM_READ
- Rename FANx_TACHO_GEN to MBFANx_TACHO_GEN
- Use standard (KiCAD) footprints for the ICs (U1-U3)
Parts:
- U1, U2: footprint SOP65P640X120-14N -> Package_SO:SOIC-14_3.9x8.7mm_P1.27mm; symbol LevelConverter SN75AHCT125:SN74AHCT125PW -> SN74AHCT125PW:SN74AHCT125PW
- U3: footprint SOIC127P600X175-16N -> Package_SO:SOIC-16_3.9x9.9mm_P1.27mm; symbol LevelConverter CD74HC4050:CD74HC4050M -> CD74HC4050M:CD74HC4050M
- U4: footprint RPi_Pico:RPi_Pico_SMD_TH -> MCU_RaspberryPi_and_Boards:RPi_Pico_SMD_TH; symbol RaspberryPi Pico:Pico -> MCU_RaspberryPi_and_Boards:Pico
Connections:
- net +3V3 renamed +3.3V
- net FAN1_PWM_READ renamed MBFAN1_PWM_READ
- net FAN1_TACHO_GEN renamed MBFAN1_TACHO_GEN
- net FAN2_PWM_READ renamed MBFAN2_PWM_READ
- net FAN2_TACHO_GEN renamed MBFAN2_TACHO_GEN
- net FAN3_PWM_READ renamed MBFAN3_PWM_READ
- net FAN3_TACHO_GEN renamed MBFAN3_TACHO_GEN
- net FAN4_PWM_READ renamed MBFAN4_PWM_READ
- net FAN4_TACHO_GEN renamed MBFAN4_TACHO_GEN
