File: boards/fanpico-0804/kicad/power.kicad_sch (KiCad schematic)
At the start: 23 parts, among them U5 SPX1117-ADJ

Commit message: PCB version 1.2
Parts:
- C5: footprint Capacitor_SMD:C_1206_3216Metric_Pad1.33x1.80mm_HandSolder -> Capacitor_Tantalum_SMD:CP_EIA-3216-18_Kemet-A_Pad1.58x1.35mm_HandSolder
- C7, C8: value 10uF 15V -> 10uF 16V; footprint Capacitor_SMD:C_1206_3216Metric_Pad1.33x1.80mm_HandSolder -> Capacitor_Tantalum_SMD:CP_EIA-3216-18_Kemet-A_Pad1.58x1.35mm_HandSolder
- R3: value 300 -> 330
Other:
- title: FanPico-0804 -> FanPico-0804 v1.2
Changed lines of the file:
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@@
   (paper "A4")
   (title_block
-    (title "FanPico-0804")
-    (date "2022-02-26")
+    (title "FanPico-0804 v1.2")
+    (date "2022-03-11")
     (company "Timo Kokkonen <tjko@iki.fi>")
-    (comment 3 "Fanpico firmware reference/prototype PCB.")
+    (comment 3 "Fanpico firmware reference PCB.")
   )
   (junction (at 175.26 29.21) (diameter 0) (color 0 0 0 0)
@@
       (effects (font (size 1.27 1.27)) (justify left))
     )
-    (property "Value" "10uF 15V" (id 1) (at 199.39 39.37 0)
-      (effects (font (size 1.27 1.27)) (justify left))
-    )
-    (property "Footprint" "Capacitor_SMD:C_1206_3216Metric_Pad1.33x1.80mm_HandSolder" (id 2) (at 196.85 39.37 0)
+    (property "Value" "10uF 16V" (id 1) (at 199.39 39.37 0)
+      (effects (font (size 1.27 1.27)) (justify left))
+    )
+    (property "Footprint" "Capacitor_Tantalum_SMD:CP_EIA-3216-18_Kemet-A_Pad1.58x1.35mm_HandSolder" (id 2) (at 196.85 39.37 0)
       (effects (font (size 1.27 1.27)) hide)
     )
@@
       (effects (font (size 1.27 1.27)) (justify left))
     )
-    (property "Value" "300" (id 1) (at 177.8 36.8299 0)
+    (property "Value" "330" (id 1) (at 177.8 36.8299 0)
       (effects (font (size 1.27 1.27)) (justify left))
     )
@@
       (effects (font (size 1.27 1.27)) (justify left))
     )
-    (property "Value" "10uF 15V" (id 1) (at 186.69 48.9838 0)
-      (effects (font (size 1.27 1.27)) (justify left))
-    )
-    (property "Footprint" "Capacitor_SMD:C_1206_3216Metric_Pad1.33x1.80mm_HandSolder" (id 2) (at 184.15 48.26 0)
+    (property "Value" "10uF 16V" (id 1) (at 186.69 48.9838 0)
+      (effects (font (size 1.27 1.27)) (justify left))
+    )
+    (property "Footprint" "Capacitor_Tantalum_SMD:CP_EIA-3216-18_Kemet-A_Pad1.58x1.35mm_HandSolder" (id 2) (at 184.15 48.26 0)
       (effects (font (size 1.27 1.27)) hide)
     )
@@
       (effects (font (size 1.27 1.27)) (justify left))
     )
-    (property "Footprint" "Capacitor_SMD:C_1206_3216Metric_Pad1.33x1.80mm_HandSolder" (id 2) (at 144.78 39.37 0)
-      (effects (font (size 1.27 1.27)) hide)
-    )
+    (property "Footprint" "Capacitor_Tantalum_SMD:CP_EIA-3216-18_Kemet-A_Pad1.58x1.35mm_HandSolder" (id 2) (at 144.78 39.37 0)
+      (effects (font (size 1.27 1.27)) hide)
+    )

Commit message: New PCB revision v1.3
Other:
- title: FanPico-0804 v1.2 -> FanPico-0804 v1.3
Changed lines of the file:
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@@
   (paper "A4")
   (title_block
-    (title "FanPico-0804 v1.2")
-    (date "2022-03-11")
+    (title "FanPico-0804 v1.3")
+    (date "2022-04-10")
     (company "Timo Kokkonen <tjko@iki.fi>")
     (comment 3 "Fanpico firmware reference PCB.")

Commit message: Cleanup schematic (no actual changes that affect PCB).
- Add labels to sub-pages so printed schematic is more readable.
- Rename FANx_PWM_READ to MBFANx_PWM_READ
- Rename FANx_TACHO_GEN to MBFANx_TACHO_GEN
- Use standard (KiCAD) footprints for the ICs (U1-U3)
Connections:
- net +3V3 renamed +3.3V
Other:
- note added: "Power Rails"
Changed lines of the file:
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@@
   (title_block
     (title "FanPico-0804 v1.3")
-    (date "2022-04-10")
+    (date "2022-08-18")
     (company "Timo Kokkonen <tjko@iki.fi>")
     (comment 3 "Fanpico firmware reference PCB.")
@@
     (stroke (width 0) (type default) (color 0 0 0 0))
   )
+  (text "Power Rails" (at 16.51 17.78 0)
+    (effects (font (size 2 2)) (justify left bottom))
+  )
   (global_label "AUX5V" (shape input) (at 63.5 177.8 180) (fields_autoplaced)
