File: boards/fanpico-0401D/kicad/fan_channel.kicad_sch (KiCad schematic)
At the start: 13 parts, among them Q1 2N7002K

Commit message: Add new 0401D v1.1 PCB (#116)
Parts:
- removed R8: 1k, Resistor_SMD:R_0603_1608Metric_Pad0.98x0.95mm_HandSolder, symbol Device:R
- added D2: 12V TVS, Diode_SMD:D_SOD-323_HandSoldering, symbol Device:D_TVS
- added D33: 5V TVS, Diode_SMD:D_SOD-323_HandSoldering, symbol Device:D_TVS
- D11: value 5V -> 5V TVS
- D15: value 12V -> 12V TVS
- D9: value BAT54C -> BAT54(C)
Connections:
- net GND: now also D2.1 (A1), D33.1 (A1)
- net PWM_OUT: now also D33.2 (A2)
- net TACHO_OUT: now also D2.2 (A2)
Other:
- title: FanPico-0401D v1.0 -> FanPico-0401D v1.1
