File: boards/fanpico-0401D/kicad/fan_channels.kicad_sch (KiCad schematic)
At the start: 8 parts, among them J12 Fan2 Output, J13 Fan3 Output, J14 Fan4 Output, J4 MB Fan1 Input, J8 Fan1 Output

Commit message: Add new 0401D v1.1 PCB (#116)
Other:
- title: FanPico-0401D v1.0 -> FanPico-0401D v1.1
Changed lines of the file:
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@@
 	(paper "A4")
 	(title_block
-		(title "FanPico-0401D v1.0")
-		(date "2024-07-22")
+		(title "FanPico-0401D v1.1")
+		(date "2024-08-15")
 		(company "Timo Kokkonen <tjko@iki.fi>")
 		(comment 3 "Fanpico firmware reference PCB.")
