File: boards/fanpico-0401D/kicad/fanpico.kicad_pcb (KiCad board)
At the start: 4 copper layers, 82.5 x 81.5 mm, 110 parts, among them J1 Floppy Power Connector, J12 Fan2 Output, J13 Fan3 Output, J14 Fan4 Output, J16 Sensor1, J17 Sensor2, J18 LCD (SPI), J19 Serial Console (TTL), J2 I2C (OLED ALT), J3 I2C (OLED)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

Commit message: Add new 0401D v1.1 PCB (#116)
Parts:
- removed R36, R39, R42: 49.9k, Resistor_SMD:R_0603_1608Metric_Pad0.98x0.95mm_HandSolder
- removed R8: 1k, Resistor_SMD:R_0603_1608Metric_Pad0.98x0.95mm_HandSolder
- removed the REF** at (66.2, 85.0)
- added D2: 12V TVS, Diode_SMD:D_SOD-323_HandSoldering, F.Cu at (91.7, 60.5)
- added D33: 5V TVS, Diode_SMD:D_SOD-323_HandSoldering, F.Cu at (104.3, 114.0)
- added D34: 5V TVS, Diode_SMD:D_SOD-323_HandSoldering, F.Cu at (104.2, 102.8)
- added D35: 5V TVS, Diode_SMD:D_SOD-323_HandSoldering, F.Cu at (104.3, 91.5)
- added D36: 5V TVS, Diode_SMD:D_SOD-323_HandSoldering, F.Cu at (104.3, 80.3)
- added JP12: 1-Wire PullUp Enable, Connector_PinHeader_2.54mm:PinHeader_1x02_P2.54mm_Vertical, F.Cu at (57.7, 120.1)
- added R2: 4.7k, Resistor_SMD:R_0603_1608Metric_Pad0.98x0.95mm_HandSolder, F.Cu at (59.4, 122.7)
- added REF**: OSHW-Logo_7.5x8mm_SilkScreen, Symbol:OSHW-Logo_7.5x8mm_SilkScreen, F.Cu at (64.4, 84.5)
- D11: value 5V -> 5V TVS
- D13, D14, D16, D17, D18, D19, D7: value 3.3V -> 3.3V TVS
- D15, D20, D21, D22: value 12V -> 12V TVS
- D23, D29: value LED 0805 (green) -> 3.3V TVS; footprint LED_SMD:LED_0805_2012Metric_Pad1.15x1.40mm_HandSolder -> Diode_SMD:D_SOD-323_HandSoldering
- D24, D27, D30, D9: value BAT54C -> BAT54(C)
- D26: value LED 0805 (green) -> 12V TVS; footprint LED_SMD:LED_0805_2012Metric_Pad1.15x1.40mm_HandSolder -> Diode_SMD:D_SOD-323_HandSoldering
- Q2: value BSS138 -> 2N7002K
- R16: value 10k -> 49.9k
- moved D26 56.9 mm to (62.7, 61.0)
- moved D23 49.5 mm to (56.4, 127.5), turned to -90 degrees
- moved D29 30.9 mm to (80.2, 68.8), turned to 0 degrees
- moved D11 7.72 mm to (93.7, 60.5), turned to -90 degrees
- moved D8 5.53 mm to (97.9, 123.1), turned to 0 degrees
- moved D12 5.19 mm to (95.9, 57.7), turned to -90 degrees
- moved R11 4.40 mm to (98.9, 60.4), turned to 0 degrees
- moved C7 4.29 mm to (62.2, 70.2), turned to 90 degrees
- moved R4 3.34 mm to (60.1, 71.3), turned to 90 degrees
- moved R3 2.80 mm to (64.2, 70.8), turned to 90 degrees
- moved R10 2.67 mm to (54.2, 70.0)
- moved Q1 2.64 mm to (99.0, 57.6)
- moved C32 1.99 mm to (80.5, 70.8)
- moved J2 1.99 mm to (84.0, 72.6)
- moved J3 1.99 mm to (84.0, 69.0)
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Connections:
- D11 pad 2: /Fan Channels/Fan1/PWM_IN -> MBFAN1_PWM_READ
- D23 pad 2: Net-(D23-A) -> 3V3
- D26 pad 2: Net-(D26-A) -> MAIN_PWR
- D29 pad 2: Net-(D29-A) -> 3V3
- J4 pad 4: /Fan Channels/Fan1/PWM_IN -> MBFAN1_PWM_READ
- R15 pad 1: +5V -> GND
Routing:
- net +5V: track 91.9 -> 58.0 mm, vias 5 -> 4
- net AGND: track 91.0 -> 122.3 mm
- net /Fan Channels/Fan1/PWM_IN: track 26.5 -> 0.00 mm
- net MAIN_PWR: track 216.2 -> 189.8 mm
- net MBFAN1_PWM_READ: track 5.32 -> 23.3 mm
- net /Power Rails/5V_REG_OUT: track 29.7 -> 18.4 mm
- net MBFAN1_TACHO_GEN: track 37.7 -> 49.0 mm
- net 3V3: track 203.9 -> 212.1 mm, vias 1 -> 0
- net SDA: track 90.1 -> 94.8 mm
- net SCL: track 84.4 -> 89.0 mm
- net Net-(U5-ADJ): track 25.8 -> 21.7 mm
- net DQ: track 37.8 -> 41.2 mm
- net /Fan Channels/Fan1/PWM_OUT: track 11.6 -> 14.8 mm
- net /Fan Channels/Fan2/PWM_OUT: track 11.6 -> 14.6 mm
- net Net-(JP12-A): track 0.00 -> 2.90 mm
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Other:
- board text added: "FanPico-0401D"
- board text added: "FanPico-0401D v1.1 by Timo Kokkonen <tjko@iki.fi> 2024-08-15"
- board text added: "MAIN POWER"
- board text added: "kokkonen.net/fanpico/"
- board text removed: "FanPico-0401D v1.0 by Timo Kokkonen <tjko@iki.fi> 2024-07-22"
- board text removed: "JLCJLC"
- board text removed: "Main Power"
- board text removed: "github.com/tjko/fanpico"
