File: boards/power-board/kicad/fanpico_powerboard.kicad_pcb (KiCad board)
At the start: 2 copper layers, 65 x 65 mm, 22 parts, among them J1 Power Input 2, J13 FANCTRL1, J14 FANCTRL2, J15 FANCTRL3, J16 FANCTRL4, J2 Power Input 1, J3 AUX Power Output, J5 FAN1, J6 FAN2, J7 FAN3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

Commit message: New version of powerboard PCB. (#130)
* Updated PCB v1.1
Routing:
- net GND: track 0.00 -> 84.7 mm, vias 3 -> 73
- net PWR: track 221.2 -> 238.5 mm
- net TACHO4: track 66.0 -> 70.7 mm
- net PWM4: track 69.1 -> 73.3 mm
- net PWM3: track 99.5 -> 103.1 mm
- net TACHO3: track 100.2 -> 103.7 mm
Other:
- board text added: "FanPico PowerBoard v1.1 by Timo Kokkonen <tjko@iki.fi> 2024-10-06"
- board text removed: "FanPico PowerBoard v1.0 by Timo Kokkonen <tjko@iki.fi> 2024-08-02"
