File: boards/fanpico-0804D/kicad/extra_fan_channel.kicad_sch (KiCad schematic)
At the start: 9 parts

Commit message: Updated schematic and design files.
Parts:
- C21: LCSC Part Number (none) -> C1588
- C22: LCSC Part Number (none) -> C1591
- D23: LCSC Part Number (none) -> C434432
- D24: LCSC Part Number (none) -> C2844172
- D25: LCSC Part Number (none) -> C445494
- R36: LCSC Part Number (none) -> C114624
- R37: LCSC Part Number (none) -> C98220
- R38: LCSC Part Number (none) -> C115415
Other:
- title: FanPico-0804D v1.1 -> FanPico-0804D v1.2
Changed lines of the file:
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@@
   (paper "A4")
   (title_block
-    (title "FanPico-0804D v1.1")
-    (date "2022-10-06")
+    (title "FanPico-0804D v1.2")
+    (date "2023-02-17")
     (company "Timo Kokkonen <tjko@iki.fi>")
     (comment 3 "Fanpico firmware reference PCB.")
@@
       (effects (font (size 1.27 1.27)) hide)
     )
+    (property "LCSC Part Number" "C1588" (id 4) (at 146.05 83.82 0)
+      (effects (font (size 1.27 1.27)) hide)
+    )
     (pin "1")
     (pin "2")
@@
       (effects (font (size 1.27 1.27)) hide)
     )
+    (property "LCSC Part Number" "C1591" (id 4) (at 167.64 125.73 0)
+      (effects (font (size 1.27 1.27)) hide)
+    )
     (pin "1")
     (pin "2")
@@
     )
     (property "Datasheet" "~" (id 3) (at 147.32 129.54 0)
+      (effects (font (size 1.27 1.27)) hide)
+    )
+    (property "LCSC Part Number" "C114624" (id 4) (at 147.32 129.54 0)
       (effects (font (size 1.27 1.27)) hide)
     )
@@
       (effects (font (size 1.27 1.27)) hide)
     )
+    (property "LCSC Part Number" "C98220" (id 4) (at 166.37 67.31 0)
+      (effects (font (size 1.27 1.27)) hide)
+    )
     (pin "1")
     (pin "2")
@@
     )
     (property "Datasheet" "~" (id 3) (at 179.07 125.73 0)
+      (effects (font (size 1.27 1.27)) hide)
+    )
+    (property "LCSC Part Number" "C445494" (id 4) (at 179.07 125.73 0)
       (effects (font (size 1.27 1.27)) hide)
     )
@@
       (effects (font (size 1.27 1.27)) hide)
     )
+    (property "LCSC Part Number" "C2844172" (id 4) (at 177.8 74.93 0)
+      (effects (font (size 1.27 1.27)) hide)
+    )
     (pin "1")
     (pin "2")
@@
       (effects (font (size 1.27 1.27)) hide)
     )
+    (property "LCSC Part Number" "C115415" (id 4) (at 167.64 46.99 0)
+      (effects (font (size 1.27 1.27)) hide)
+    )
     (pin "1")
     (pin "2")
@@
       (effects (font (size 1.27 1.27)) hide)
     )
+    (property "LCSC Part Number" "C434432" (id 4) (at 147.32 139.7 0)
+      (effects (font (size 1.27 1.27)) hide)
+    )

Commit message: Updated 0804D PCB v1.2c
Parts:
- D24: footprint Diode_SMD:D_SOT-23_ANK -> FanPico:D_SOT-23_ANK
Other:
- title: FanPico-0804D v1.2 -> FanPico-0804D v1.2(c)

Commit message: New FanPico-0804D PCB v1.3
Parts:
- added D53: 12V TVS, Diode_SMD:D_SOD-323_HandSoldering, symbol Device:D_TVS_Small
- added D69: 5V TVS, Diode_SMD:D_SOD-323_HandSoldering, symbol Device:D_TVS_Small
- renumbered C21 to C23, C22 to C24, D23 to D26, D24 to D27, D25 to D28, JP6 to JP7, R36 to R39, R37 to R40, R38 to R41
Connections:
- net GND: now also D53.1 (A1), D69.1 (A1)
- net PWM_OUT: now also D69.2 (A2)
- net TACHO_IN: now also D53.2 (A2)
Other:
- title: FanPico-0804D v1.2(c) -> FanPico-0804D v1.3b
