File: boards/fanpico-0804D/kicad/fan_channel.kicad_sch (KiCad schematic)
At the start: 16 parts, among them Q1 2N7002K

Commit message: Updated schematic and design files.
Parts:
- C10: LCSC Part Number (none) -> C1588
- C11: LCSC Part Number (none) -> C1591
- D10: LCSC Part Number (none) -> C445494
- D7, D8: LCSC Part Number (none) -> C434432
- D9: LCSC Part Number (none) -> C2844172
- Q1: LCSC Part Number (none) -> C85047
- R10, R12: LCSC Part Number (none) -> C114624
- R11, R8: LCSC Part Number (none) -> C22548
- R13: LCSC Part Number (none) -> C98220
- R14: LCSC Part Number (none) -> C115415
- R9: LCSC Part Number (none) -> C100001
Connections:
- net +3.3V: no longer R9.2
- net GND: now also R9.1
- net PWM_READ: now also R9.2; no longer R9.1
Other:
- title: FanPico-0804D v1.1 -> FanPico-0804D v1.2
- moved on the sheet: R9
Changed lines of the file:
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@@
   (paper "A4")
   (title_block
-    (title "FanPico-0804D v1.1")
-    (date "2022-10-06")
+    (title "FanPico-0804D v1.2")
+    (date "2023-02-17")
     (company "Timo Kokkonen <tjko@iki.fi>")
     (comment 3 "Fanpico firmware reference PCB.")
@@
     (stroke (width 0) (type default) (color 0 0 0 0))
   )
+  (wire (pts (xy 105.41 43.18) (xy 105.41 49.53))
+    (stroke (width 0) (type default) (color 0 0 0 0))
+  )
   (wire (pts (xy 205.74 43.18) (xy 229.87 43.18))
     (stroke (width 0) (type default) (color 0 0 0 0))
@@
     (stroke (width 0) (type default) (color 0 0 0 0))
   )
-  (wire (pts (xy 105.41 26.67) (xy 115.57 26.67))
-    (stroke (width 0) (type default) (color 0 0 0 0))
-  )
   (wire (pts (xy 97.79 43.18) (xy 105.41 43.18))
     (stroke (width 0) (type default) (color 0 0 0 0))
@@
     (stroke (width 0) (type default) (color 0 0 0 0))
   )
+  (wire (pts (xy 105.41 57.15) (xy 105.41 59.69))
+    (stroke (width 0) (type default) (color 0 0 0 0))
+  )
   (polyline (pts (xy 224.79 31.75) (xy 224.79 144.78))
     (stroke (width 0) (type default) (color 0 0 0 0))
@@
     (stroke (width 0) (type default) (color 0 0 0 0))
   )
-  (wire (pts (xy 105.41 38.1) (xy 105.41 43.18))
-    (stroke (width 0) (type default) (color 0 0 0 0))
-  )
   (wire (pts (xy 171.45 71.12) (xy 190.5 71.12))
     (stroke (width 0) (type default) (color 0 0 0 0))
@@
   )
   (wire (pts (xy 190.5 139.7) (xy 190.5 144.78))
-    (stroke (width 0) (type default) (color 0 0 0 0))
-  )
-  (wire (pts (xy 105.41 30.48) (xy 105.41 26.67))
     (stroke (width 0) (type default) (color 0 0 0 0))
   )
@@
     (effects (font (size 1.27 1.27)) (justify right))
   )
-  (symbol (lib_id "Device:R") (at 105.41 34.29 180) (unit 1)
-    (in_bom yes) (on_board yes) (fields_autoplaced)
-    (property "Reference" "R9" (id 0) (at 107.95 33.0199 0)
-      (effects (font (size 1.27 1.27)) (justify right))
-    )
-    (property "Value" "30k" (id 1) (at 107.95 35.5599 0)
-      (effects (font (size 1.27 1.27)) (justify right))
-    )
-    (property "Footprint" "Resistor_SMD:R_0603_1608Metric_Pad0.98x0.95mm_HandSolder" (id 2) (at 107.188 34.29 90)
-      (effects (font (size 1.27 1.27)) hide)
-    )
-    (property "Datasheet" "~" (id 3) (at 105.41 34.29 0)
+  (symbol (lib_id "Device:R") (at 105.41 53.34 180) (unit 1)
+    (in_bom yes) (on_board yes) (fields_autoplaced)
+    (property "Reference" "R9" (id 0) (at 107.95 52.0699 0)
+      (effects (font (size 1.27 1.27)) (justify right))
+    )
+    (property "Value" "30k" (id 1) (at 107.95 54.6099 0)
+      (effects (font (size 1.27 1.27)) (justify right))
+    )
+    (property "Footprint" "Resistor_SMD:R_0603_1608Metric_Pad0.98x0.95mm_HandSolder" (id 2) (at 107.188 53.34 90)
+      (effects (font (size 1.27 1.27)) hide)
+    )
+    (property "Datasheet" "~" (id 3) (at 105.41 53.34 0)
+      (effects (font (size 1.27 1.27)) hide)
+    )
+    (property "LCSC Part Number" "C100001" (id 4) (at 105.41 53.34 0)
       (effects (font (size 1.27 1.27)) hide)
     )
@@
     )
     (property "Datasheet" "~" (id 3) (at 190.5 125.73 0)
+      (effects (font (size 1.27 1.27)) hide)
+    )
+    (property "LCSC Part Number" "C114624" (id 4) (at 190.5 125.73 0)
       (effects (font (size 1.27 1.27)) hide)
     )
@@
       (effects (font (size 1.27 1.27)) hide)
     )
+    (property "LCSC Part Number" "C2844172" (id 4) (at 212.09 71.12 0)
+      (effects (font (size 1.27 1.27)) hide)
+    )
     (pin "1")
     (pin "2")
@@
       (effects (font (size 1.27 1.27)) hide)
     )
+    (property "LCSC Part Number" "C22548" (id 4) (at 93.98 43.18 0)
+      (effects (font (size 1.27 1.27)) hide)
+    )
     (pin "1")
     (pin "2")
@@
       (effects (font (size 1.27 1.27)) (justify left) hide)
     )
+    (property "LCSC Part Number" "C85047" (id 4) (at 104.14 88.9 0)
+      (effects (font (size 1.27 1.27)) hide)
+    )
     (pin "1")
     (pin "2")
     (pin "3")
   )
-  (symbol (lib_id "power:+3.3V") (at 115.57 26.67 270) (unit 1)
-    (in_bom yes) (on_board yes) (fields_autoplaced)
-    (property "Reference" "#PWR036" (id 0) (at 111.76 26.67 0)
-      (effects (font (size 1.27 1.27)) hide)
-    )
-    (property "Value" "+3.3V" (id 1) (at 119.38 26.6699 90)
-      (effects (font (size 1.27 1.27)) (justify left))
-    )
-    (property "Footprint" "" (id 2) (at 115.57 26.67 0)
-      (effects (font (size 1.27 1.27)) hide)
-    )
-    (property "Datasheet" "" (id 3) (at 115.57 26.67 0)
-      (effects (font (size 1.27 1.27)) hide)
-    )
-    (pin "1")
-  )
   (symbol (lib_id "Device:C") (at 190.5 80.01 0) (unit 1)
     (in_bom yes) (on_board yes) (fields_autoplaced)
@@
     )
     (property "Datasheet" "~" (id 3) (at 190.5 80.01 0)
+      (effects (font (size 1.27 1.27)) hide)
+    )
+    (property "LCSC Part Number" "C1588" (id 4) (at 190.5 80.01 0)
       (effects (font (size 1.27 1.27)) hide)
     )
@@
       (effects (font (size 1.27 1.27)) hide)
     )
+    (property "LCSC Part Number" "C22548" (id 4) (at 116.84 80.01 0)
+      (effects (font (size 1.27 1.27)) hide)
+    )
     (pin "1")
     (pin "2")
@@
       (effects (font (size 1.27 1.27)) (justify right))
     )
-    (property "Value" "LED 0805 (green)" (id 1) (at 179.07 138.43 90)
+    (property "Value" "LED 0805 (green)" (id 1) (at 171.45 139.7 90)
       (effects (font (size 1.27 1.27)) (justify right))
     )
@@
     )
     (property "Datasheet" "~" (id 3) (at 190.5 135.89 0)
+      (effects (font (size 1.27 1.27)) hide)
+    )
+    (property "LCSC Part Number" "C434432" (id 4) (at 190.5 135.89 0)
       (effects (font (size 1.27 1.27)) hide)
     )
@@
       (effects (font (size 1.27 1.27)) hide)
     )
+    (property "LCSC Part Number" "C98220" (id 4) (at 200.66 63.5 0)
+      (effects (font (size 1.27 1.27)) hide)
+    )
     (pin "1")
     (pin "2")
@@
       (effects (font (size 1.27 1.27)) hide)
     )
+    (property "LCSC Part Number" "C445494" (id 4) (at 215.9 125.73 0)
+      (effects (font (size 1.27 1.27)) hide)
+    )
     (pin "1")
     (pin "2")
@@
       (effects (font (size 1.27 1.27)) hide)
     )
+    (property "LCSC Part Number" "C1591" (id 4) (at 204.47 125.73 0)
+      (effects (font (size 1.27 1.27)) hide)
+    )
     (pin "1")
     (pin "2")
@@
       (effects (font (size 1.27 1.27)) hide)
     )
+    (property "LCSC Part Number" "C114624" (id 4) (at 107.95 139.7 0)
+      (effects (font (size 1.27 1.27)) hide)
+    )
     (pin "1")
     (pin "2")
@@
     )
     (property "Datasheet" "~" (id 3) (at 107.95 149.86 0)
+      (effects (font (size 1.27 1.27)) hide)
+    )
+    (property "LCSC Part Number" "C434432" (id 4) (at 107.95 149.86 0)
       (effects (font (size 1.27 1.27)) hide)
     )
@@
       (effects (font (size 1.27 1.27)) hide)
     )
-    (pin "1")
-    (pin "2")
+    (property "LCSC Part Number" "C115415" (id 4) (at 201.93 43.18 0)
+      (effects (font (size 1.27 1.27)) hide)
+    )
+    (pin "1")
+    (pin "2")
+  )
+  (symbol (lib_id "power:GND") (at 105.41 59.69 0) (unit 1)
+    (in_bom yes) (on_board yes) (fields_autoplaced)
+    (property "Reference" "#PWR037" (id 0) (at 105.41 66.04 0)
+      (effects (font (size 1.27 1.27)) hide)
+    )
+    (property "Value" "GND" (id 1) (at 105.41 64.77 0))
+    (property "Footprint" "" (id 2) (at 105.41 59.69 0)
+      (effects (font (size 1.27 1.27)) hide)
+    )
+    (property "Datasheet" "" (id 3) (at 105.41 59.69 0)
+      (effects (font (size 1.27 1.27)) hide)
+    )
+    (pin "1")
   )
 )

Commit message: Updated 0804D PCB v1.2c
Parts:
- D9: footprint Diode_SMD:D_SOT-23_ANK -> FanPico:D_SOT-23_ANK
Other:
- title: FanPico-0804D v1.2 -> FanPico-0804D v1.2(c)

Commit message: New FanPico-0804D PCB v1.3
Parts:
- removed TP6: TestPoint, TestPoint:TestPoint_Pad_D1.5mm, symbol Connector:TestPoint
- added D46, D50, D62: 12V TVS, Diode_SMD:D_SOD-323_HandSoldering, symbol Device:D_TVS_Small
- added D58, D66: 5V TVS, Diode_SMD:D_SOD-323_HandSoldering, symbol Device:D_TVS_Small
- renumbered C10 to C19, C11 to C20, D7 to D19, D8 to D20, D9 to D21, D10 to D22, JP2 to JP5, Q1 to Q4, R8 to R29, R9 to R30, R10 to R31, R11 to R32, R12 to R33, R13 to R34, R14 to R35
Connections:
- net GND: now also D46.1 (A1), D50.1 (A1), D58.1 (A1), D62.1 (A1), D66.1 (A1)
- net PWM_IN: now also D58.2 (A2)
- net PWM_OUT: now also D66.2 (A2)
- net PWR_IN: now also D46.2 (A2)
- net TACHO_IN: now also D50.2 (A2)
- net TACHO_OUT: now also D62.2 (A2)
Other:
- title: FanPico-0804D v1.2(c) -> FanPico-0804D v1.3b
