File: boards/fanpico-0804D/kicad/fan_channels.kicad_sch (KiCad schematic)
At the start: 12 parts, among them J10 Fan3 Output, J11 Fan4 Output, J12 Fan5 Output, J13 Fan6 Output, J14 Fan7 Output, J15 Fan8 Output, J4 MB Fan1 Input, J5 MB Fan2 Input, J6 MB Fan3 Input, J7 MB Fan4 Input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

Commit message: Updated schematic and design files.
Other:
- title: FanPico-0804D v1.1 -> FanPico-0804D v1.2
Changed lines of the file:
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@@
   (paper "A4")
   (title_block
-    (title "FanPico-0804D v1.1")
-    (date "2022-10-06")
+    (title "FanPico-0804D v1.2")
+    (date "2023-02-17")
     (company "Timo Kokkonen <tjko@iki.fi>")
     (comment 3 "Fanpico firmware reference PCB.")

Commit message: Updated 0804D PCB v1.2c
Other:
- title: FanPico-0804D v1.2 -> FanPico-0804D v1.2(c)

Commit message: New FanPico-0804D PCB v1.3
Other:
- title: FanPico-0804D v1.2(c) -> FanPico-0804D v1.3b
