File: boards/fanpico-0804D/kicad/fanpico.kicad_pcb (KiCad board)
At the start: 2 copper layers, 135 x 81.5 mm, 173 parts, among them J1 Floppy Power Connector, J10 Fan3 Output, J11 Fan4 Output, J12 Fan5 Output, J13 Fan6 Output, J14 Fan7 Output, J15 Fan8 Output, J16 Sensor1, J17 Sensor2, J18 SPI (Future Use), J19 Serial Console (TTL), J3 I2C (OLED), J4 MB Fan1 Input, J5 MB Fan2 Input, J6 MB Fan3 Input, J7 MB Fan4 Input, J8 Fan1 Output, J9 Fan2 Output, Q1 2N7002K, Q2 2N7002K, Q3 2N7002K, Q4 2N7002K, SW1 SW_Push, U1 SN74AHCT125QDRQ1, U2 SN74AHCT125QDRQ1, U3 CD74HC4050NSR, U4 Pico, U5 SPX1117-ADJ, U6 LM4040DBZ-3, U7 74HC4051

Commit message: Updated schematic and design files.
Parts:
- added J2: I2C (OLED ALT), Connector_PinSocket_2.54mm:PinSocket_1x04_P2.54mm_Vertical, F.Cu at (117.7, 80.9)
- added REF**: ToolingHole_1.152mm, FanPico:ToolingHole_1.152mm, F.Cu at (163.5, 133.5)
- added REF**: ToolingHole_1.152mm, FanPico:ToolingHole_1.152mm, F.Cu at (46.5, 133.5)
- added REF**: ToolingHole_1.152mm, FanPico:ToolingHole_1.152mm, F.Cu at (46.5, 56.0)
- J18: value SPI (Future Use) -> LCD (SPI); footprint Connector_PinHeader_2.54mm:PinHeader_2x03_P2.54mm_Vertical -> Connector_PinHeader_2.54mm:PinHeader_2x05_P2.54mm_Vertical
- moved R1 13.8 mm to (63.7, 62.2)
- moved SW1 1.71 mm to (58.5, 62.2)
- moved D12 1.40 mm to (115.9, 113.1)
- moved D8 1.40 mm to (104.7, 113.1)
- moved D16 1.30 mm to (138.4, 113.0)
- moved D20 1.30 mm to (127.4, 113.0)
- moved REF** 1.10 mm to (158.1, 122.5)
- moved C32 0.98 mm to (114.2, 79.1), turned to 180 degrees
- moved C5 0.95 mm to (69.5, 77.2)
- moved TP8 0.88 mm to (124.7, 71.9)
- moved R19 0.60 mm to (115.9, 116.0)
- moved R26 0.57 mm to (138.8, 116.0)
- moved R12 0.56 mm to (104.9, 116.0)
- moved R33 0.55 mm to (127.2, 116.0)
- moved J19 0.50 mm to (43.4, 119.9)
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Connections:
- C4 pad 1: /VSYS -> VSYS
- D1 pad 1: /VSYS -> VSYS
- R16 pad 1: MBFAN2_PWM_READ -> GND
- R16 pad 2: 3V3 -> MBFAN2_PWM_READ
- R23 pad 1: MBFAN4_PWM_READ -> GND
- R23 pad 2: 3V3 -> MBFAN4_PWM_READ
- R30 pad 1: MBFAN3_PWM_READ -> GND
- R30 pad 2: 3V3 -> MBFAN3_PWM_READ
- R9 pad 1: MBFAN1_PWM_READ -> GND
- R9 pad 2: 3V3 -> MBFAN1_PWM_READ
- U4 pad 39: /VSYS -> VSYS
Routing:
- net VSYS: track 0.00 -> 72.3 mm
- net 3V3: track 493.0 -> 462.8 mm, vias 23 -> 17
- net /VSYS: track 13.9 -> 0.00 mm
- net RESET: track 42.2 -> 31.7 mm
- net GND: track 206.8 -> 197.0 mm, vias 88 -> 90
- net SDA_SCK: track 122.9 -> 127.8 mm
- net FAN5_PWM_GEN: track 112.8 -> 117.2 mm
- net SCL_MOSI: track 115.9 -> 119.7 mm
- net TEMP1_READ: track 64.7 -> 62.6 mm
- net TEMP2_READ: track 88.3 -> 86.1 mm
- net FAN3_PWR: track 133.2 -> 131.4 mm
- net Net-(R1-Pad2): track 9.01 -> 10.8 mm
- net TX_MISO: track 27.0 -> 28.6 mm
- net Net-(D16-Pad2): track 3.74 -> 2.57 mm
- net Net-(D20-Pad2): track 3.31 -> 2.22 mm
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Other:
- outline, holes or cut-outs redrawn
- board text added: "0804D v1.2"
- board text added: "BL"
- board text added: "DC"
- board text added: "FanPico-0804D v1.2 by Timo Kokkonen <tjko@iki.fi> 2023-02-17"
- board text added: "LCD (SPI)"
- board text added: "RST"
- board text removed: "0804D v1.1"
- board text removed: "FanPico-0804D v1.1 by Timo Kokkonen <tjko@iki.fi> 2022-10-04"
- board text removed: "MISO"
- board text removed: "SPI"

Commit message: Updated 0804D PCB v1.2c
Parts:
- removed the REF** at (163.5, 133.5)
- removed the REF** at (46.5, 133.5)
- removed the REF** at (46.5, 56.0)
- added R54: DNF, Resistor_SMD:R_0603_1608Metric_Pad0.98x0.95mm_HandSolder, F.Cu at (63.9, 119.0)
- added R55: 0, Resistor_SMD:R_0603_1608Metric_Pad0.98x0.95mm_HandSolder, F.Cu at (63.9, 117.4)
- added R56: DNF, Resistor_SMD:R_0603_1608Metric_Pad0.98x0.95mm_HandSolder, F.Cu at (74.4, 119.0)
- added R57: 0, Resistor_SMD:R_0603_1608Metric_Pad0.98x0.95mm_HandSolder, F.Cu at (74.4, 117.4)
- C5: value 10uF 20V -> 10uF 25V; footprint Capacitor_Tantalum_SMD:CP_EIA-3216-18_Kemet-A_Pad1.58x1.35mm_HandSolder -> Capacitor_Tantalum_SMD:CP_EIA-3528-12_Kemet-T_Pad1.50x2.35mm_HandSolder
- D13, D17, D21, D24, D27, D30, D33, D9: footprint Diode_SMD:D_SOT-23_ANK -> FanPico:D_SOT-23_ANK
- J1: footprint Connector_TE-Connectivity:TE 171826-4 Floppy 4-pin -> FanPico:TE 171826-4 Floppy 4-pin
- SW1: footprint Button_Switch_THT:SW_PUSH_6mm_SMD_2 -> FanPico:SW_PUSH_6mm_SMD_2
- U1, U2: value SN74AHCT125QDRQ1 -> SN74AHCT126
- moved D3 4.41 mm to (70.7, 71.0), turned to 90 degrees
- moved C6 3.64 mm to (79.5, 72.0), turned to 90 degrees
- moved U5 3.64 mm to (84.2, 74.8)
- moved C31 2.03 mm to (98.3, 77.1), turned to 180 degrees
- moved C5 0.29 mm to (69.7, 77.4)
- turned D4 to 0 degrees
Connections:
- net Net-(C5-Pad1) renamed /Power Rails/5V_REG_IN
- net Net-(C8-Pad1) renamed /Power Rails/5V_REG_OUT
- net Net-(D3-Pad2) renamed /Power Rails/5V_REG_SEL
- net Net-(F1-Pad1) renamed /Sensors & Connectors/AUX12_IN
- U1 pad 1: GND -> Net-(U1-~{1OE})
- U1 pad 10: GND -> Net-(U1-~{1OE})
- U1 pad 13: GND -> Net-(U1-~{1OE})
- U1 pad 4: GND -> Net-(U1-~{1OE})
- U2 pad 1: GND -> Net-(U2-~{1OE})
- U2 pad 10: GND -> Net-(U2-~{1OE})
- U2 pad 13: GND -> Net-(U2-~{1OE})
- U2 pad 4: GND -> Net-(U2-~{1OE})
Routing:
- net Net-(U1-~{1OE}): track 0.00 -> 36.8 mm, vias 0 -> 2
- net Net-(U2-~{1OE}): track 0.00 -> 36.2 mm, vias 0 -> 2
- net GND: track 197.0 -> 169.4 mm, vias 90 -> 95
- net +5V: track 101.4 -> 107.9 mm
- net /Power Rails/5V_REG_SEL: track 9.84 -> 3.77 mm
- net Net-(U5-ADJ): track 32.2 -> 27.9 mm
- net /Power Rails/5V_REG_OUT: track 24.2 -> 20.2 mm
- net /Power Rails/5V_REG_IN: track 19.6 -> 16.5 mm
- net FAN6_PWM_GEN: track 110.4 -> 113.3 mm
- net 3V3: track 462.8 -> 460.0 mm
- net /PWM4B: track 23.2 -> 20.5 mm
- net MBFAN2_TACHO_GEN: track 79.8 -> 78.6 mm
- net SDA_SCK: track 127.8 -> 126.5 mm
- net Net-(D4-A): track 3.07 -> 4.24 mm
- net SCL_MOSI: track 119.7 -> 118.6 mm
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Other:
- board text added: "FanPico-0804D v1.2(c) by Timo Kokkonen <tjko@iki.fi> 2024-01-02"
- board text added: "JLCJLC"
- board text removed: "0804D v1.2"
- board text removed: "FanPico-0804D v1.2 by Timo Kokkonen <tjko@iki.fi> 2023-02-17"

Commit message: New FanPico-0804D PCB v1.3
Parts:
- removed the REF** at (158.1, 122.5)
- removed TP1, TP2, TP3, TP4, TP5, TP6, TP7, TP8, TP9: TestPoint, TestPoint:TestPoint_Pad_D1.5mm
- added D35: LED 0805 (green), LED_SMD:LED_0805_2012Metric_Pad1.15x1.40mm_HandSolder, F.Cu at (68.3, 58.2)
- added D36: 3.3V TVS, Diode_SMD:D_SOD-323_HandSoldering, F.Cu at (50.6, 80.5)
- added D37: 3.3V TVS, Diode_SMD:D_SOD-323_HandSoldering, F.Cu at (50.6, 78.5)
- added D38: 3.3V TVS, Diode_SMD:D_SOD-323_HandSoldering, F.Cu at (47.0, 121.0)
- added D39: 3.3V TVS, Diode_SMD:D_SOD-323_HandSoldering, F.Cu at (47.0, 126.2)
- added D40: 3.3V TVS, Diode_SMD:D_SOD-323_HandSoldering, F.Cu at (113.8, 78.3)
- added D41: 3.3V TVS, Diode_SMD:D_SOD-323_HandSoldering, F.Cu at (132.5, 77.7)
- added D42: 3.3V TVS, Diode_SMD:D_SOD-323_HandSoldering, F.Cu at (132.5, 75.6)
- added D43: 12V TVS, Diode_SMD:D_SOD-323_HandSoldering, F.Cu at (61.5, 66.0)
- added D44: 12V TVS, Diode_SMD:D_SOD-323_HandSoldering, F.Cu at (100.4, 64.9)
- added D45: 12V TVS, Diode_SMD:D_SOD-323_HandSoldering, F.Cu at (112.1, 65.0)
- added D46: 12V TVS, Diode_SMD:D_SOD-323_HandSoldering, F.Cu at (123.6, 65.0)
- added D47: 12V TVS, Diode_SMD:D_SOD-323_HandSoldering, F.Cu at (135.1, 65.0)
- added D48: 12V TVS, Diode_SMD:D_SOD-323_HandSoldering, F.Cu at (108.7, 114.5)
- added D49: 12V TVS, Diode_SMD:D_SOD-323_HandSoldering, F.Cu at (119.7, 114.7)
- added D50: 12V TVS, Diode_SMD:D_SOD-323_HandSoldering, F.Cu at (131.0, 114.7)
- added D51: 12V TVS, Diode_SMD:D_SOD-323_HandSoldering, F.Cu at (145.4, 128.7)
- added D52: 12V TVS, Diode_SMD:D_SOD-323_HandSoldering, F.Cu at (152.9, 107.8)
- added D53: 12V TVS, Diode_SMD:D_SOD-323_HandSoldering, F.Cu at (152.9, 96.4)
- added D54: 12V TVS, Diode_SMD:D_SOD-323_HandSoldering, F.Cu at (152.8, 84.0)
- added D55: 12V TVS, Diode_SMD:D_SOD-323_HandSoldering, F.Cu at (152.9, 74.4)
- added D56: 5V TVS, Diode_SMD:D_SOD-323_HandSoldering, F.Cu at (108.3, 66.4)
- added D57: 5V TVS, Diode_SMD:D_SOD-323_HandSoldering, F.Cu at (119.9, 66.5)
- added D58: 5V TVS, Diode_SMD:D_SOD-323_HandSoldering, F.Cu at (131.7, 66.5)
- added D59: 5V TVS, Diode_SMD:D_SOD-323_HandSoldering, F.Cu at (143.6, 66.5)
- added D60: 12V TVS, Diode_SMD:D_SOD-323_HandSoldering, F.Cu at (104.5, 64.9)
- added D61: 12V TVS, Diode_SMD:D_SOD-323_HandSoldering, F.Cu at (116.2, 65.0)
- added D62: 12V TVS, Diode_SMD:D_SOD-323_HandSoldering, F.Cu at (127.8, 65.0)
- added D63: 12V TVS, Diode_SMD:D_SOD-323_HandSoldering, F.Cu at (139.3, 65.0)
- added D64: 5V TVS, Diode_SMD:D_SOD-323_HandSoldering, F.Cu at (102.2, 115.3)
- added D65: 5V TVS, Diode_SMD:D_SOD-323_HandSoldering, F.Cu at (112.3, 115.3)
- added D66: 5V TVS, Diode_SMD:D_SOD-323_HandSoldering, F.Cu at (123.5, 115.3)
- added D67: 5V TVS, Diode_SMD:D_SOD-323_HandSoldering, F.Cu at (134.9, 115.2)
- added D68: 5V TVS, Diode_SMD:D_SOD-323_HandSoldering, F.Cu at (152.8, 113.1)
- added D69: 5V TVS, Diode_SMD:D_SOD-323_HandSoldering, F.Cu at (150.4, 99.5)
- added D70: 5V TVS, Diode_SMD:D_SOD-323_HandSoldering, F.Cu at (150.1, 88.7)
- added D71: 5V TVS, Diode_SMD:D_SOD-323_HandSoldering, F.Cu at (149.9, 77.7)
- added D72: 3.3V TVS, Diode_SMD:D_SOD-323_HandSoldering, F.Cu at (50.3, 125.9)
- added D73: 3.3V TVS, Diode_SMD:D_SOD-323_HandSoldering, F.Cu at (51.7, 120.9)
- added D74: 3.3V TVS, Diode_SMD:D_SOD-323_HandSoldering, F.Cu at (49.3, 121.0)
- added G1: qwiic_Logo, sparkfun-qwiic:qwiic_5mm, F.Cu at (50.6, 128.2)
- added J20: 1-Wire, TerminalBlock_TE-Connectivity:TerminalBlock_TE_282834-3_1x03_P2.54mm_Horizontal, F.Cu at (44.8, 84.8)
- added J21: QWIIC, Connector_JST:JST_SH_SM04B-SRSS-TB_1x04-1MP_P1.00mm_Horizontal, F.Cu at (50.6, 132.2)
- added JP12: 1-Wire Pull-Up Enable, Connector_PinHeader_2.54mm:PinHeader_1x02_P2.54mm_Vertical, F.Cu at (54.6, 78.2)
- added R58: 49.9k, Resistor_SMD:R_0603_1608Metric_Pad0.98x0.95mm_HandSolder, F.Cu at (72.0, 58.0)
- added R59: 4.7k, Resistor_SMD:R_0603_1608Metric_Pad0.98x0.95mm_HandSolder, F.Cu at (54.5, 81.8)
- added REF**: Symbol_Barrel_Polarity, Symbol:Symbol_Barrel_Polarity, F.Cu at (54.3, 68.6)
- added REF**: OSHW-Logo_7.5x8mm_SilkScreen, Symbol:OSHW-Logo_7.5x8mm_SilkScreen, F.Cu at (158.3, 120.4)
- J1: value Floppy Power Connector -> Floppy / DC Connector; footprint FanPico:TE 171826-4 Floppy 4-pin -> FanPico:TE 171826-4 Floppy 4-pin Combo
- U5: footprint Package_TO_SOT_SMD:SOT-223 -> Package_TO_SOT_SMD:SOT-223-3_TabPin2
- moved SW1 115.2 mm to (153.0, 128.0), turned to 0 degrees
- moved R1 108.8 mm to (148.6, 130.2), turned to 90 degrees
- moved R5 31.3 mm to (59.2, 61.2)
- moved D4 31.2 mm to (59.1, 58.1), turned to 180 degrees
- moved D6 25.6 mm to (50.1, 58.2), turned to 180 degrees
- moved R7 25.4 mm to (49.9, 61.2)
- moved D5 20.9 mm to (54.7, 58.2)
- moved R6 20.1 mm to (54.8, 61.2), turned to 180 degrees
- moved D1 16.3 mm to (62.6, 75.3)
- moved D2 9.50 mm to (63.4, 58.2)
- moved C4 8.84 mm to (42.2, 77.0), turned to 180 degrees
- moved R2 6.22 mm to (63.4, 61.2)
- moved J18 5.05 mm to (57.3, 119.8)
- moved R54 4.94 mm to (68.8, 119.0)
- moved R55 4.94 mm to (68.8, 117.4)
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Connections:
- J1 pad 1: AUX5V -> unconnected-(J1-Pin_1-Pad1)
- U6 pad 3: (no net) -> unconnected-(U6-NC-Pad3)
Routing:
- net RESET: track 31.7 -> 126.2 mm
- net TX_MISO: track 28.6 -> 108.5 mm
- net SCL_MOSI: track 118.6 -> 168.9 mm
- net SDA_SCK: track 126.5 -> 164.8 mm
- net VSYS: track 72.3 -> 109.1 mm, vias 0 -> 1
- net 3V3: track 460.0 -> 483.6 mm
- net VBUS: track 18.4 -> 38.4 mm
- net /Sensors & Connectors/AUX12_IN: track 13.1 -> 27.1 mm
- net RX_CS: track 22.5 -> 34.7 mm, vias 1 -> 0
- net AUX12V: track 204.0 -> 194.6 mm
- net /Power Rails/5V_REG_SEL: track 3.77 -> 12.2 mm
- net FAN7_PWM_GEN: track 112.6 -> 104.2 mm
- net FAN6_PWM_GEN: track 113.3 -> 105.4 mm
- net FAN1_PWM_GEN: track 71.8 -> 64.6 mm
- net MBFAN3_PWM_READ: track 103.8 -> 110.6 mm
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Other:
- board text added: "+"
- board text added: "-"
- board text added: "1-WIRE"
- board text added: "12V 3A"
- board text added: "DQ"
- board text added: "FanPico-0804D"
- board text added: "FanPico-0804D v1.3(b) by Timo Kokkonen <tjko@iki.fi> 2024-08-29"
- board text added: "MAIN"
- board text added: "USB"
- board text added: "VDD"
- board text added: "kokkonen.net/fanpico/"
- board text removed: "12V (AUX)"
- board text removed: "FanPico-0804D v1.2(c) by Timo Kokkonen <tjko@iki.fi> 2024-01-02"
- board text removed: "JLCJLC"
- board text removed: "USB Power"
- board text removed: "github.com/tjko/fanpico"
