File: boards/fanpico-0804D/kicad/fanpico.kicad_sch (KiCad schematic)
At the start: 22 parts, among them SW1 SW_Push, U1 SN74AHCT125QDRQ1, U2 SN74AHCT125QDRQ1, U3 CD74HC4050NSR, U4 Pico, U6 LM4040DBZ-3, U7 74HC4051

Commit message: Updated schematic and design files.
Parts:
- removed D1: SM5819PL 1A 40V, Diode_SMD:D_SMA, symbol Device:D_Schottky
- C1, C2, C29, C3, C31, C4: LCSC Part Number (none) -> C1591
- C30: LCSC Part Number (none) -> C7171
- R1: LCSC Part Number (none) -> C22548
- R48: LCSC Part Number (none) -> C105881
- R49: LCSC Part Number (none) -> C100044
- U1, U2: LCSC Part Number (none) -> C155176
- U3: LCSC Part Number (none) -> C131932
- U6: LCSC Part Number (none) -> C143326
- U7: LCSC Part Number (none) -> C9386
Other:
- sheet Sensors renamed Sensors & Connectors
- title: FanPico-0804D v1.1 -> FanPico-0804D v1.2

Commit message: Updated 0804D PCB v1.2c
Parts:
- added R54, R56: DNF, Resistor_SMD:R_0603_1608Metric_Pad0.98x0.95mm_HandSolder, symbol Device:R
- added R55, R57: 0, Resistor_SMD:R_0603_1608Metric_Pad0.98x0.95mm_HandSolder, symbol Device:R
- R49: LCSC Part Number C100044 -> C21189
- SW1: footprint Button_Switch_THT:SW_PUSH_6mm_SMD_2 -> FanPico:SW_PUSH_6mm_SMD_2
- U1, U2: value SN74AHCT125QDRQ1 -> SN74AHCT126; symbol SN74AHCT125PW:SN74AHCT125PW -> fanpico:SN74AHCT125PW; LCSC Part Number C155176 -> C163728
- U3: symbol CD74HC4050M:CD74HC4050M -> fanpico:CD74HC4050NSR
- U4: symbol MCU_RaspberryPi_and_Boards:Pico -> fanpico:Pico
Connections:
- net +5V: now also R55.1, R57.1
- net GND: now also R54.1, R56.1; no longer U1.1 (~{1OE}), U1.10 (~{3OE}), U1.13 (~{4OE}), U1.4 (~{2OE}), U2.1 (~{1OE}), U2.10 (~{3OE}), U2.13 (~{4OE}), U2.4 (~{2OE})
- new net: R56.2, R57.2, U2.1 (~{1OE}), U2.10 (~{3OE}), U2.13 (~{4OE}), U2.4 (~{2OE})
- new net: R54.2, R55.2, U1.1 (~{1OE}), U1.10 (~{3OE}), U1.13 (~{4OE}), U1.4 (~{2OE})
Other:
- title: FanPico-0804D v1.2 -> FanPico-0804D v1.2(c)

Commit message: New FanPico-0804D PCB v1.3
Parts:
- added G1: qwiic_Logo, sparkfun-qwiic:qwiic_5mm, symbol sprakfun-qwiic:qwiic_Logo
- H1, H2, H3, H4: now not fitted
- R54, R56: value DNF -> 0; LCSC Part Number (none) -> C21189; now not fitted
- SW1: LCSC Part Number (none) -> C221880
Other:
- title: FanPico-0804D v1.2(c) -> FanPico-0804D v1.3b
