File: boards/fanpico-0804D/kicad/power.kicad_sch (KiCad schematic)
At the start: 23 parts, among them U5 SPX1117-ADJ

Commit message: Updated schematic and design files.
Parts:
- added D1: SM5819PL 1A 40V, Diode_SMD:D_SMA, symbol Device:D_Schottky
- C5: LCSC Part Number (none) -> C117023
- C6: LCSC Part Number (none) -> C1591
- C7, C8: LCSC Part Number (none) -> C7171
- D2, D4, D5, D6: LCSC Part Number (none) -> C434432
- D3: LCSC Part Number (none) -> C445494
- F2: LCSC Part Number (none) -> C70072
- R2: LCSC Part Number (none) -> C114624
- R3: LCSC Part Number (none) -> C105881
- R4: LCSC Part Number (none) -> C22548
- R5, R7: LCSC Part Number (none) -> C98220
- R6: LCSC Part Number (none) -> C114621
- U5: LCSC Part Number (none) -> C67402
Connections:
- net +5V: now also D1.2 (A)
- new net VSYS: D1.1 (K)
Other:
- title: FanPico-0804D v1.1 -> FanPico-0804D v1.2
- moved on the sheet: C5, C6, C7, C8, D2, D3, D4, F2, JP1, R2, R3, R4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

Commit message: Updated 0804D PCB v1.2c
Parts:
- C5: value 10uF 20V -> 10uF 25V; footprint Capacitor_Tantalum_SMD:CP_EIA-3216-18_Kemet-A_Pad1.58x1.35mm_HandSolder -> Capacitor_Tantalum_SMD:CP_EIA-3528-12_Kemet-T_Pad1.50x2.35mm_HandSolder; LCSC Part Number C117023 -> C7194
- U5: symbol Regulator_Linear:LM1117-ADJ -> Regulator_Linear:AP1117-ADJ
Connections:
- net 5V_REG_IN: now reaches C5.1, C6.1, D3.1 (K), U5.3 (VI)
- net 5V_REG_SEL: now reaches D3.2 (A), JP1.2 (C)
- net 5V_REG_OUT: now reaches C8.1, F2.1, R3.1, U5.2 (VO)
Other:
- title: FanPico-0804D v1.2 -> FanPico-0804D v1.2(c)
- moved on the sheet: JP1

Commit message: New FanPico-0804D PCB v1.3
Parts:
- removed TP1, TP2, TP3, TP4, TP5: TestPoint, TestPoint:TestPoint_Pad_D1.5mm, symbol Connector:TestPoint
- added D35: LED 0805 (green), LED_SMD:LED_0805_2012Metric_Pad1.15x1.40mm_HandSolder, symbol Device:LED
- added R58: 49.9k, Resistor_SMD:R_0603_1608Metric_Pad0.98x0.95mm_HandSolder, symbol Device:R
- D1: LCSC Part Number C669023 -> C669023 or C19992592
- U5: footprint Package_TO_SOT_SMD:SOT-223 -> Package_TO_SOT_SMD:SOT-223-3_TabPin2
Connections:
- net 5V_REG_SEL: now also R58.1
- net GND: now also D35.1 (K)
- new net: D35.2 (A), R58.2
Other:
- title: FanPico-0804D v1.2(c) -> FanPico-0804D v1.3b
