File: boards/fanpico-0804D/kicad/sensors.kicad_sch (KiCad schematic)
At the start: 14 parts, among them J1 Floppy Power Connector, J16 Sensor1, J17 Sensor2, J18 SPI (Future Use), J19 Serial Console (TTL), J3 I2C (OLED)

Commit message: Updated schematic and design files.
Parts:
- added J2: I2C (OLED ALT), Connector_PinSocket_2.54mm:PinSocket_1x04_P2.54mm_Vertical, symbol Connector_Generic:Conn_01x04
- C32: LCSC Part Number (none) -> C1591
- F1: LCSC Part Number (none) -> C20829
- J18: value SPI (Future Use) -> LCD (SPI); footprint Connector_PinHeader_2.54mm:PinHeader_2x03_P2.54mm_Vertical -> Connector_PinHeader_2.54mm:PinHeader_2x05_P2.54mm_Vertical; symbol Connector_Generic:Conn_02x03_Odd_Even -> Connector_Generic:Conn_02x05_Odd_Even
- R50, R51: LCSC Part Number (none) -> C98220
- R52, R53: LCSC Part Number (none) -> C14675
Connections:
- net +3.3V: now also J18.7 (Pin_7), J18.8 (Pin_8), J2.1 (Pin_1)
- net GND: now also J18.10 (Pin_10), J2.2 (Pin_2)
- net SCL_MOSI: now also J2.3 (Pin_3)
- net SDA_SCK: now also J2.4 (Pin_4)
- new net VSYS: J18.9 (Pin_9)
Other:
- title: FanPico-0804D v1.1 -> FanPico-0804D v1.2
- moved on the sheet: J19

Commit message: Updated 0804D PCB v1.2c
Parts:
- F1: LCSC Part Number C20829 -> C2977527
- J1: footprint Connector_TE-Connectivity:TE 171826-4 Floppy 4-pin -> FanPico:TE 171826-4 Floppy 4-pin
Connections:
- net AUX12_IN: now reaches F1.1, J1.4 (Pin_4)
Other:
- title: FanPico-0804D v1.2 -> FanPico-0804D v1.2(c)
- moved on the sheet: F1, J1

Commit message: New FanPico-0804D PCB v1.3
Parts:
- added D36, D37, D38, D39, D40, D41, D42, D72, D73, D74: 3.3V TVS, Diode_SMD:D_SOD-323_HandSoldering, symbol Device:D_TVS_Small
- added D43: 12V TVS, Diode_SMD:D_SOD-323_HandSoldering, symbol Device:D_TVS_Small
- added J20: 1-Wire, TerminalBlock_TE-Connectivity:TerminalBlock_TE_282834-3_1x03_P2.54mm_Horizontal, symbol Connector_Generic:Conn_01x03
- added J21: QWIIC, Connector_JST:JST_SH_SM04B-SRSS-TB_1x04-1MP_P1.00mm_Horizontal, symbol Connector_Generic:Conn_01x04
- added JP12: 1-Wire Pull-Up Enable, Connector_PinHeader_2.54mm:PinHeader_1x02_P2.54mm_Vertical, symbol Jumper:Jumper_2_Open
- added R59: 4.7k, Resistor_SMD:R_0603_1608Metric_Pad0.98x0.95mm_HandSolder, symbol Device:R
- J1: value Floppy Power Connector -> Floppy / DC Connector; footprint FanPico:TE 171826-4 Floppy 4-pin -> FanPico:TE 171826-4 Floppy 4-pin Combo; LCSC Part Number (none) -> C590635 / C720558
Connections:
- net +3.3V: now also D37.2 (A2), D40.2 (A2), D72.2 (A2), J20.3 (Pin_3), J21.2 (Pin_2), R59.2
- net AUX12_IN: now also D43.2 (A2)
- net GND: now also D36.1 (A1), D37.1 (A1), D38.1 (A1), D39.1 (A1), D40.1 (A1), D41.1 (A1), D42.1 (A1), D43.1 (A1), D72.1 (A1), D73.1 (A1), D74.1 (A1), J20.1 (Pin_1), J21.1 (Pin_1)
- net RX_CS: now also D38.2 (A2)
- net SCL_MOSI: now also D41.2 (A2), D73.2 (A2), J21.4 (Pin_4)
- net SDA_SCK: now also D42.2 (A2), D74.2 (A2), J21.3 (Pin_3)
- net TX_MISO: now also D36.2 (A2), D39.2 (A2), J20.2 (Pin_2), JP12.1 (A)
- net AUX5V: no longer names the net of J1.1 (Pin_1)
- new net: JP12.2 (B), R59.1
- no-connect marks 0 -> 1
Other:
- note added: "1-Wire Bus shares pins with Serial (This can't be used if Serial or SPI is in use)"
- title: FanPico-0804D v1.2(c) -> FanPico-0804D v1.3b
- moved on the sheet: C32, F1, J1, J16, J17, J18, J19, J2, J3, JP10, JP11, R50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
